Commit message: update config for Borunte

File: src/borunte_support/urdf/borunte_stand_macro.xacro (robot description, xacro)
@@ -26,5 +26,5 @@
                 <child link="${prefix}borunte_stand_flange"/>
                 <axis xyz="0 0 0"/>
-                <origin rpy="0.0 0.0 -0.785398163" xyz="-0.1591 0.1591 0.70485"/>
+                <origin rpy="0.0 0.0 -0.719" xyz="0.053 -0.053 0.719"/>
         </joint>
 </xacro:macro>

Commit message: borunte_robot: correct robot stand position

File: src/borunte_support/urdf/borunte_stand_macro.xacro (robot description, xacro)
@@ -26,5 +26,5 @@
                 <child link="${prefix}borunte_stand_flange"/>
                 <axis xyz="0 0 0"/>
-                <origin rpy="0.0 0.0 -0.719" xyz="0.053 -0.053 0.719"/>
+                <origin rpy="0.0 0.0 ${pi/4.0}" xyz="0.053 0.053 0.719"/>
         </joint>
 </xacro:macro>

Commit message: borunte_support: fix misaligned stand

File: src/borunte_support/urdf/borunte_stand_macro.xacro (robot description, xacro)
@@ -2,9 +2,9 @@
 <robot xmlns:xacro="http://www.ros.org/wiki/xacro">
 <xacro:macro name="borunte_stand" params="prefix">
-        <!-- link list -->
+        <!-- link list  -->
 	    <link name="${prefix}borunte_stand_link">
                 <visual>
                         <geometry>
-                                <mesh filename="package://borunte_support/meshes/stand-urdf-prototype.stl"/>
+                                <mesh filename="package://borunte_support/meshes/borunte_carriage.stl"/>
                         </geometry>
                         <origin rpy="0.0 0 0.0" xyz="0 0 0"/>
@@ -15,7 +15,7 @@
                 <collision>
                         <geometry>
-                                <mesh filename="package://borunte_support/meshes/stand-urdf-prototype.stl"/>
+                                <mesh filename="package://borunte_support/meshes/borunte_carriage.stl"/>
                         </geometry>
-                        <origin rpy="0.0 0 0.0" xyz="0 0 0"/>
+                        <origin rpy="0.0 0 0.0" xyz="0 0 0.016"/>
                 </collision>
         </link>
@@ -26,5 +26,5 @@
                 <child link="${prefix}borunte_stand_flange"/>
                 <axis xyz="0 0 0"/>
-                <origin rpy="0.0 0.0 ${pi/4.0}" xyz="0.053 0.053 0.719"/>
+                <origin rpy="0.0 0.0 ${pi/4.0}" xyz="0.0 0.0 0.735"/>
         </joint>
 </xacro:macro>

Commit message: introduce world reference frame

File: src/borunte_support/urdf/borunte_stand_macro.xacro (robot description, xacro)
@@ -20,4 +20,12 @@
       </collision>
     </link>
+    <!-- 'world' frame: default pose reference frame -->
+    <link name="${prefix}world" />
+    <joint name="${prefix}rb07_stand_link-world" type="fixed">
+      <origin xyz="0 0 0" rpy="0 0 0"/>
+      <axis xyz="0 0 1"/>
+      <parent link="${prefix}borunte_stand_link"/>
+      <child link="${prefix}world"/>
+    </joint>
     <!-- link the robot is going to be attached to -->
     <link name="${prefix}borunte_stand_flange" />
