Commit message: borunte_support: fix Robotiq Gripper dimensions

File: src/borunte_support/urdf/borunte_hand_e_fish_fingers_macro.xacro (robot description, xacro)
@@ -18,5 +18,5 @@
     <joint name="${prefix}flange-tool0" type="fixed">
       <!-- marker -->
-      <origin xyz="0.0468199 0.0 0.157234" rpy="0 ${pi*5/4} 0" />
+      <origin xyz="0.0468199 0.0 0.158734" rpy="0 ${pi*5/4} 0" />
       <parent link="${prefix}flange" />
       <child link="${prefix}tool0" />
@@ -26,5 +26,5 @@
     <joint name="${prefix}flange-tool1" type="fixed">
       <!-- marker -->
-      <origin xyz="-0.119652 0.0 0.228652" rpy="0 ${pi*3/4} 0" />
+      <origin xyz="-0.119652 0.0 0.230152" rpy="0 ${pi*3/4} 0" />
       <parent link="${prefix}flange" />
       <child link="${prefix}tool1" />

File: src/borunte_support/urdf/borunte_hand_e_macro.xacro (robot description, xacro)
@@ -18,5 +18,5 @@
     <joint name="${prefix}flange-tool0" type="fixed">
       <!-- marker -->
-      <origin xyz="0 0 0.159" rpy="0 ${pi*1} 0" />
+      <origin xyz="0 0 0.1605" rpy="0 ${pi*1} 0" />
       <parent link="${prefix}flange" />
       <child link="${prefix}tool0" />

File: src/borunte_support/urdf/robotiq_hand_e_base_macro.xacro (robot description, xacro)
@@ -28,5 +28,5 @@
           <mesh filename="package://borunte_support/meshes/robotiq_hand-e_gripper.stl"/>
         </geometry>
-        <origin xyz="0 0 -0.005" rpy="0 0 0"/>
+        <origin xyz="0 0 -0.003" rpy="0 0 0"/>
         <material name="Black_Aluminum"/>
       </visual>

File: src/borunte_support/urdf/robotiq_hand_e_fish_fingers_macro.xacro (robot description, xacro)
@@ -26,5 +26,5 @@
       <child link="${prefix}fish_finger_adapter_left" />
       <axis xyz="0 0 1"/>
-      <origin xyz="0 0 0.095" rpy="0 0 ${pi/2.0}" />
+      <origin xyz="0 0 0.0965" rpy="0 0 ${pi/2.0}" />
     </joint>
     <link name="${prefix}fish_finger_adapter_right">
@@ -47,5 +47,5 @@
       <child link="${prefix}fish_finger_adapter_right" />
       <axis xyz="0 0 1"/>
-      <origin xyz="0 0 0.095" rpy="0 0 -${pi/2.0}" />
+      <origin xyz="0 0 0.0965" rpy="0 0 -${pi/2.0}" />
     </joint>
     <link name="${prefix}simple_grip_finger_left">

File: src/borunte_support/urdf/robotiq_hand_e_macro.xacro (robot description, xacro)
@@ -23,5 +23,5 @@
       <child link="${prefix}simple_grip_finger_left" />
       <axis xyz="0 0 1"/>
-      <origin xyz="0 0 0.095" rpy="0 0 ${pi/2.0}" />
+      <origin xyz="0 0 0.0965" rpy="0 0 ${pi/2.0}" />
     </joint>
     <link name="${prefix}simple_grip_finger_right">
@@ -44,5 +44,5 @@
       <child link="${prefix}simple_grip_finger_right" />
       <axis xyz="0 0 1"/>
-      <origin xyz="0 0 0.095" rpy="0 0 -${pi/2.0}" />
+      <origin xyz="0 0 0.0965" rpy="0 0 -${pi/2.0}" />
     </joint>
   </xacro:macro>

Commit message: borunte_support: simplify fish fingers

File: src/borunte_support/urdf/borunte_hand_e_fish_fingers_macro.xacro (robot description, xacro)
@@ -18,15 +18,21 @@
     <joint name="${prefix}flange-tool0" type="fixed">
       <!-- marker -->
-      <origin xyz="0.0468199 0.0 0.158734" rpy="0 ${pi*5/4} 0" />
+      <origin xyz="0.0 0.0 0.0" rpy="0 ${pi*1} 0" />
       <parent link="${prefix}flange" />
       <child link="${prefix}tool0" />
     </joint>
-    <!-- ROS-Industrial 'tool1' frame: all-zeros tool frame -->
-    <link name="${prefix}tool1" />
-    <joint name="${prefix}flange-tool1" type="fixed">
+    <link name="${prefix}eef_tcp_simple_grip" />
+    <joint name="${prefix}flange-eef_tcp_simple_grip" type="fixed">
+      <!-- marker -->
+      <origin xyz="0.0468199 0.0 0.158734" rpy="0 ${pi*5/4} 0" />
+      <parent link="${prefix}flange" />
+      <child link="${prefix}eef_tcp_simple_grip" />
+    </joint>
+    <link name="${prefix}eef_tcp_fish_grip" />
+    <joint name="${prefix}flange-eef_tcp_fish_grip" type="fixed">
       <!-- marker -->
       <origin xyz="-0.119652 0.0 0.230152" rpy="0 ${pi*3/4} 0" />
       <parent link="${prefix}flange" />
-      <child link="${prefix}tool1" />
+      <child link="${prefix}eef_tcp_fish_grip" />
     </joint>
   </xacro:macro>

Commit message: borunte_support: move camera frame definition to tool init

File: src/borunte_support/urdf/borunte_hand_e_fish_fingers_macro.xacro (robot description, xacro)
@@ -13,4 +13,11 @@
       <parent link="${prefix}flange" />
       <child link="${prefix}borunte_robotiq_adapter" />
+    </joint>
+      <!-- Camera frame: location of wrist camera -->
+    <link name="${prefix}rgb_camera_link" />
+    <joint name="${prefix}borunte_robotiq_adapter-rgb_camera_link" type="fixed">
+      <origin xyz="0.06 0 0.03" rpy="0 0 ${pi/2.0}" />
+      <parent link="${prefix}borunte_robotiq_adapter" />
+      <child link="${prefix}rgb_camera_link" />
     </joint>
     <!-- ROS-Industrial 'tool0' frame: all-zeros tool frame -->

File: src/borunte_support/urdf/borunte_hand_e_macro.xacro (robot description, xacro)
@@ -14,4 +14,11 @@
       <child link="${prefix}borunte_robotiq_adapter" />
     </joint>
+    <!-- Camera frame: location of wrist camera -->
+    <link name="${prefix}rgb_camera_link" />
+    <joint name="${prefix}borunte_robotiq_adapter-rgb_camera_link" type="fixed">
+      <origin xyz="0.06 0 0.03" rpy="0 0 ${pi/2.0}" />
+      <parent link="${prefix}borunte_robotiq_adapter" />
+      <child link="${prefix}rgb_camera_link" />
+    </joint>
     <!-- ROS-Industrial 'tool0' frame: all-zeros tool frame -->
     <link name="${prefix}tool0" />

File: src/borunte_support/urdf/robotiq_hand_e_base_macro.xacro (robot description, xacro)
@@ -44,11 +44,4 @@
       <origin xyz="0 0 0.015" rpy="${pi} ${pi} ${pi/2.0}" />
     </joint>
-    <!-- Camera frame: location of wrist camera -->
-    <link name="${prefix}rgb_camera_link" />
-    <joint name="${prefix}borunte_robotiq_adapter-rgb_camera_link" type="fixed">
-      <origin xyz="0.06 0 0.03" rpy="0 0 ${pi/2.0}" />
-      <parent link="${prefix}borunte_robotiq_adapter" />
-      <child link="${prefix}rgb_camera_link" />
-    </joint>
     </xacro:macro>
 </robot>
