Commit message: borunte_robot: add fish finger gripper

File: src/borunte_support/urdf/borunte_on_stand_macro.xacro (robot description, xacro)
@@ -8,4 +8,8 @@
     <xacro:if value="${tool == 'hand_e'}">
       <xacro:include filename="$(find borunte_support)/urdf/borunte_hand_e_macro.xacro"/>
+      <xacro:borunte_hand_e_macro prefix="${robotprefix}"/>
+    </xacro:if>
+    <xacro:if value="${tool == 'hand_e_fish_fingers'}">
+      <xacro:include filename="$(find borunte_support)/urdf/borunte_hand_e_fish_fingers_macro.xacro"/>
       <xacro:borunte_hand_e_macro prefix="${robotprefix}"/>
     </xacro:if>

File: src/borunte_support/urdf/robotiq_hand_e_macro.xacro (robot description, xacro)
@@ -2,46 +2,6 @@
 <robot xmlns:xacro="http://www.ros.org/wiki/xacro">
   <xacro:macro name="robotiq_hand_e_macro" params="prefix">
-    <material name="Black_Aluminum">
-      <color rgba="0.1 0.1 0.1 1.0"/>
-    </material>
-    <material name="White_Plastic">
-      <color rgba="0.9 0.9 0.9 1.0"/>
-    </material>
-    <link name="${prefix}borunte_robotiq_adapter">
-      <visual>
-        <geometry>
-          <mesh filename="package://borunte_support/meshes/robotiq_adapter.stl"/>
-        </geometry>
-        <origin xyz="0 0 0" rpy="0 0 0" />
-        <material name="White_Plastic"/>
-      </visual>
-      <collision>
-        <geometry>
-          <mesh filename="package://borunte_support/meshes/robotiq_adapter_collision.stl"/>
-        </geometry>
-        <origin xyz="0 0 0" rpy="0 0 0" />
-      </collision>
-    </link>
-    <link name="${prefix}robotiq_hand_e">
-      <visual>
-        <geometry>
-          <mesh filename="package://borunte_support/meshes/robotiq_hand-e_gripper.stl"/>
-        </geometry>
-        <origin xyz="0 0 -0.005" rpy="0 0 0"/>
-        <material name="Black_Aluminum"/>
-      </visual>
-      <collision>
-        <geometry>
-          <mesh filename="package://borunte_support/meshes/robotiq_hand-e_gripper_collision.stl"/>
-        </geometry>
-        <origin xyz="0 0 0" rpy="0 0 0"/>
-      </collision>
-    </link>
-    <joint name="${prefix}borunte_robotiq_adapter-robotiq_hand_e" type="fixed">
-      <parent link="${prefix}borunte_robotiq_adapter" />
-      <child link="${prefix}robotiq_hand_e" />
-      <axis xyz="0 0 1"/>
-      <origin xyz="0 0 0.015" rpy="${pi} ${pi} ${pi/2.0}" />
-    </joint>
+    <xacro:include filename="$(find borunte_support)/urdf/robotiq_hand_e_base_macro.xacro"/>
+    <xacro:robotiq_hand_e_base_macro prefix="${prefix}"/>
     <link name="${prefix}simple_grip_finger_left">
       <visual>
@@ -86,11 +46,4 @@
       <origin xyz="0 0 0.095" rpy="0 0 -${pi/2.0}" />
     </joint>
-    <!-- Camera frame: location of wrist camera -->
-    <link name="${prefix}camera_link" />
-    <joint name="${prefix}borunte_robotiq_adapter-camera_link" type="fixed">
-      <origin xyz="0.06 0 0.03" rpy="0 0 ${pi/2.0}" />
-      <parent link="${prefix}borunte_robotiq_adapter" />
-      <child link="${prefix}camera_link" />
-    </joint>
   </xacro:macro>
 </robot>

Commit message: borunte_robot: cleanup URDFs

File: src/borunte_support/urdf/borunte_on_stand_macro.xacro (robot description, xacro)
@@ -21,5 +21,5 @@
     <xacro:borunte_stand_macro prefix="${standprefix}"/>
     <!-- attach robot to stand flange -->
-    <joint name="robot_attach_joint" type="fixed">
+    <joint name="${robotprefix}robot_attach_joint" type="fixed">
       <parent link="borunte_stand_flange"/>
       <child link="${robotprefix}base_link"/>

File: src/borunte_support/urdf/borunte_stand_macro.xacro (robot description, xacro)
@@ -2,4 +2,7 @@
 <robot xmlns:xacro="http://ros.org/wiki/xacro">
   <xacro:macro name="borunte_stand_macro" params="prefix">
+    <material name="DarkGray">
+      <color rgba="0.5 0.5 0.5 1.0"/>
+    </material>
     <!-- link list  -->
     <link name="${prefix}borunte_stand_link">
@@ -9,7 +12,5 @@
         </geometry>
         <origin rpy="0.0 0 0.0" xyz="0 0 0"/>
-        <material name="DarkGray">
-          <color rgba="0.5 0.5 0.5 1.0"/>
-        </material>
+        <material name="DarkGray"/>
       </visual>
       <collision>
@@ -17,10 +18,10 @@
           <mesh filename="package://borunte_support/meshes/borunte_carriage.stl"/>
         </geometry>
-        <origin rpy="0.0 0 0.0" xyz="0 0 0.016"/>
+        <origin rpy="0.0 0 0.0" xyz="0 0 0.0"/>
       </collision>
     </link>
     <!-- 'world' frame: default pose reference frame -->
     <link name="${prefix}world" />
-    <joint name="${prefix}rb07_stand_link-world" type="fixed">
+    <joint name="${prefix}borunte_stand_link-world" type="fixed">
       <origin xyz="0 0 0" rpy="0 0 0"/>
       <axis xyz="0 0 1"/>
