Commit message: borunte_support: fix ezgrippr tool offset

File: src/borunte_support/urdf/borunte_ezgripper_gen2_plus_macro.xacro (robot description, xacro)
@@ -46,5 +46,5 @@
     <joint name="${prefix}flange-tool0" type="fixed">
       <!-- marker -->
-      <origin xyz="0 0 0.183" rpy="0 ${pi*1} ${-pi/2.0}" />
+      <origin xyz="0 0 0.195" rpy="0 ${pi*1} ${-pi/2.0}" />
       <parent link="${prefix}flange" />
       <child link="${prefix}tool0" />

Commit message: borunte_support: use new camera names

File: src/borunte_support/urdf/borunte_ezgripper_gen2_plus_macro.xacro (robot description, xacro)
@@ -27,10 +27,16 @@
       </collision>
     </link>
-    <!-- Camera frame: location of wrist camera -->
-    <link name="${prefix}camera_link" />
-    <joint name="${prefix}borunte_ezgripper_adapter-camera_link" type="fixed">
-      <origin xyz="0.06 0 0.03" rpy="0 0 ${pi/2.0}" />
+    <!-- Camera frame: location of wrist cameras -->
+    <link name="${prefix}rgb_camera_link" />
+    <joint name="${prefix}borunte_ezgripper_adapter-rgb_camera_link" type="fixed">
+      <origin xyz="0.0391 0 0.082" rpy="0 0 ${pi/2.0}" />
       <parent link="${prefix}borunte_ezgripper_adapter" />
-      <child link="${prefix}camera_link" />
+      <child link="${prefix}rgb_camera_link" />
+    </joint>
+    <link name="${prefix}depth_camera_link" />
+    <joint name="${prefix}borunte_ezgripper_adapter-depth_camera_link" type="fixed">
+      <origin xyz="-0.0321 0 0.0885" rpy="0 0 ${pi/2.0}" />
+      <parent link="${prefix}borunte_ezgripper_adapter" />
+      <child link="${prefix}depth_camera_link" />
     </joint>
     <!-- attach hand_e to eef -->

File: src/borunte_support/urdf/robotiq_hand_e_base_macro.xacro (robot description, xacro)
@@ -45,9 +45,9 @@
     </joint>
     <!-- Camera frame: location of wrist camera -->
-    <link name="${prefix}camera_link" />
-    <joint name="${prefix}borunte_robotiq_adapter-camera_link" type="fixed">
+    <link name="${prefix}rgb_camera_link" />
+    <joint name="${prefix}borunte_robotiq_adapter-rgb_camera_link" type="fixed">
       <origin xyz="0.06 0 0.03" rpy="0 0 ${pi/2.0}" />
       <parent link="${prefix}borunte_robotiq_adapter" />
-      <child link="${prefix}camera_link" />
+      <child link="${prefix}rgb_camera_link" />
     </joint>
     </xacro:macro>

Commit message: borunte_support: correcting camera position

File: src/borunte_support/urdf/borunte_ezgripper_gen2_plus_macro.xacro (robot description, xacro)
@@ -30,5 +30,5 @@
     <link name="${prefix}rgb_camera_link" />
     <joint name="${prefix}borunte_ezgripper_adapter-rgb_camera_link" type="fixed">
-      <origin xyz="0.0391 0 0.082" rpy="0 0 ${pi/2.0}" />
+      <origin xyz="0.0391 0 0.0885" rpy="0 0 ${pi/2.0}" />
       <parent link="${prefix}borunte_ezgripper_adapter" />
       <child link="${prefix}rgb_camera_link" />

Commit message: brounte_support: mount cameras on ezgripper adapter

File: src/borunte_support/urdf/borunte_ezgripper_gen2_plus_macro.xacro (robot description, xacro)
@@ -4,5 +4,5 @@
     <xacro:include filename="$(find borunte_support)/urdf/borunte_macro.xacro"/>
     <xacro:borunte_macro prefix="${prefix}"/>
-    <xacro:include filename="$(find ezgripper_driver)/urdf/ezgripper_dual_gen2_plus_cam_articulated.urdf.xacro"/>
+    <xacro:include filename="$(find ezgripper_driver)/urdf/ezgripper_dual_gen2_plus_articulated.urdf.xacro"/>
     <!-- Add the gripper -->
     <ezgripper_dual prefix="main" parent_link="${prefix}borunte_ezgripper_adapter">
@@ -30,5 +30,5 @@
     <link name="${prefix}rgb_camera_link" />
     <joint name="${prefix}borunte_ezgripper_adapter-rgb_camera_link" type="fixed">
-      <origin xyz="0.0391 0 0.0885" rpy="0 0 ${pi/2.0}" />
+      <origin xyz="0.042 0 0.052" rpy="0 0 ${pi/2.0}" />
       <parent link="${prefix}borunte_ezgripper_adapter" />
       <child link="${prefix}rgb_camera_link" />
@@ -36,5 +36,5 @@
     <link name="${prefix}depth_camera_link" />
     <joint name="${prefix}borunte_ezgripper_adapter-depth_camera_link" type="fixed">
-      <origin xyz="-0.0321 0 0.0885" rpy="0 0 ${pi/2.0}" />
+      <origin xyz="0.074 0 0.0325" rpy="0 0 ${pi/2.0}" />
       <parent link="${prefix}borunte_ezgripper_adapter" />
       <child link="${prefix}depth_camera_link" />

Commit message: use 13MP ELP camera module and fix camera positions

File: src/borunte_support/urdf/borunte_ezgripper_gen2_plus_macro.xacro (robot description, xacro)
@@ -30,5 +30,5 @@
     <link name="${prefix}rgb_camera_link" />
     <joint name="${prefix}borunte_ezgripper_adapter-rgb_camera_link" type="fixed">
-      <origin xyz="0.042 0 0.052" rpy="0 0 ${pi/2.0}" />
+      <origin xyz="0.042 0 0.027" rpy="0 0 ${pi/2.0}" />
       <parent link="${prefix}borunte_ezgripper_adapter" />
       <child link="${prefix}rgb_camera_link" />
@@ -36,5 +36,5 @@
     <link name="${prefix}depth_camera_link" />
     <joint name="${prefix}borunte_ezgripper_adapter-depth_camera_link" type="fixed">
-      <origin xyz="0.074 0 0.0325" rpy="0 0 ${pi/2.0}" />
+      <origin xyz="0.074 0 0.0255" rpy="0 0 ${pi/2.0}" />
       <parent link="${prefix}borunte_ezgripper_adapter" />
       <child link="${prefix}depth_camera_link" />

Commit message: borunte_robot: rotate ezgripper around

File: src/borunte_support/urdf/borunte_ezgripper_gen2_plus_macro.xacro (robot description, xacro)
@@ -7,5 +7,5 @@
     <!-- Add the gripper -->
     <ezgripper_dual prefix="main" parent_link="${prefix}borunte_ezgripper_adapter">
-      <origin xyz="0 0 0.012" rpy="${pi} ${-pi/2.0} 0.0"/>
+      <origin xyz="0 0 0.012" rpy="${pi} ${-pi/2.0} 0"/>
     </ezgripper_dual>
     <material name="Black_Plastic">
@@ -44,5 +44,5 @@
     <!-- this assures that planning is done from the perspective of the fingers -->
     <joint name="${prefix}flange-borunte_ezgripper_adapter" type="fixed">
-      <origin xyz="0 0 0" rpy="0 0 0" />
+      <origin xyz="0 0 0" rpy="0 0 ${pi}" />
       <parent link="${prefix}flange" />
       <child link="${prefix}borunte_ezgripper_adapter" />
