Commit message: change URDF model color

File: src/borunte_support/urdf/borunte_macro.xacro (robot description, xacro)
@@ -9,6 +9,6 @@
                         </geometry>
                         <origin rpy="0.0 0 0.0" xyz="0 0 0"/>
-                        <material name="DarkGray">
-                                <color rgba="0.5 0.5 0.5 1.0"/>
+                        <material name="Black">
+                                <color rgba="0.1 0.1 0.1 1.0"/>
                         </material>
                 </visual>
@@ -26,6 +26,6 @@
                         </geometry>
                         <origin rpy="0.0 0 0.0" xyz="0 0 0"/>
-                        <material name="DarkGray">
-                                <color rgba="0.5 0.5 0.5 1.0"/>
+                        <material name="DarkRed">
+                                <color rgba="0.5 0.0 0.0 1.0"/>
                         </material>
                 </visual>
@@ -47,7 +47,5 @@
                         </geometry>
                         <origin rpy="0.0 0 0.0" xyz="0 0 0"/>
-                        <material name="DarkGray">
-                                <color rgba="0.5 0.5 0.5 1.0"/>
-                        </material>
+                        <material name="DarkRed"/>
                 </visual>
                 <collision>
@@ -68,7 +66,5 @@
                         </geometry>
                         <origin rpy="0.0 0 0.0" xyz="0 0 0"/>
-                        <material name="DarkGray">
-                                <color rgba="0.5 0.5 0.5 1.0"/>
-                        </material>
+                        <material name="DarkRed"/>
                 </visual>
                 <collision>
@@ -89,7 +85,5 @@
                         </geometry>
                         <origin rpy="0.0 0.0 0.0" xyz="0 0 0"/>
-                        <material name="DarkGray">
-                                <color rgba="0.5 0.5 0.5 1.0"/>
-                        </material>
+                        <material name="DarkRed"/>
                 </visual>
                 <collision>
@@ -110,7 +104,5 @@
                         </geometry>
                         <origin rpy="0 0 0" xyz="0 0 0"/>
-                        <material name="DarkGray">
-                                <color rgba="0.5 0.5 0.5 1.0"/>
-                        </material>
+                        <material name="DarkRed"/>
                 </visual>
                 <collision>
@@ -131,7 +123,5 @@
                         </geometry>
                         <origin rpy="0 0 0.0" xyz="0 0 0"/>
-                        <material name="DarkGray">
-                                <color rgba="0.5 0.5 0.5 1.0"/>
-                        </material>
+                        <material name="DarkRed"/>
                 </visual>
                 <collision>

Commit message: update URDF positions

File: src/borunte_support/urdf/borunte_macro.xacro (robot description, xacro)
@@ -156,5 +156,5 @@
                 <child link="link_3"/>
                 <axis xyz="0 1 0"/>
-                <origin rpy="0.0 ${pi/2.0} 0.0" xyz="0.0 0.0 0.390"/>
+                <origin rpy="0.0 ${pi/2.0} 0.0" xyz="0.0 0.0 0.39"/>
         </joint>
 	<joint name="${prefix}joint_4" type="revolute">
@@ -163,5 +163,5 @@
                 <child link="link_4"/>
                 <axis xyz="0 0 1"/>
-                <origin rpy="0.0 0.0 0.0" xyz="-0.125 -0.0955 0.0950"/>
+                <origin rpy="0.0 0.0 0.0" xyz="-0.125 -0.1 0.095"/>
         </joint>
         <joint name="${prefix}joint_5" type="revolute">
@@ -170,5 +170,5 @@
                 <child link="link_5"/>
                 <axis xyz="0 1 0"/>
-                <origin rpy="0.0 0.0 0.0" xyz="0.0 -0.0 0.29"/>
+                <origin rpy="0.0 0.0 0.0" xyz="0.0 -0.0 0.3095"/>
         </joint>
 	<joint name="${prefix}joint_6" type="revolute">

Commit message: borunte_config: increase movement range

File: src/borunte_support/urdf/borunte_macro.xacro (robot description, xacro)
@@ -145,5 +145,5 @@
         </joint>
 	<joint name="${prefix}joint_2" type="revolute">
-		<limit effort="1000.0" lower="-1.571" upper="1.571" velocity="1.0"/>
+		<limit effort="1000.0" lower="-1.74" upper="2.35" velocity="1.0"/>
                 <parent link="link_1"/>
                 <child link="link_2"/>

Commit message: borunte_robot: add gripper to urdf

File: src/borunte_support/urdf/borunte_macro.xacro (robot description, xacro)
@@ -173,5 +173,5 @@
         </joint>
 	<joint name="${prefix}joint_6" type="revolute">
-                <limit effort="1000.0" lower="-3.141" upper="3.141" velocity="2.35"/>
+                <limit effort="1000.0" lower="${-pi}" upper="${pi}" velocity="2.35"/>
                 <parent link="link_5"/>
                 <child link="link_6"/>
@@ -195,9 +195,30 @@
         </joint>
         <!-- ROS-Industrial 'tool0' frame: all-zeros tool frame -->
-        <link name="${prefix}tool0" />
+        <link name="${prefix}tool0">
+            <visual>
+                    <geometry>
+                        <mesh filename="package://borunte_support/meshes/robotiq_gripper.stl"/>
+                    </geometry>
+                    <origin rpy="0 0 0.0" xyz="0 0 0"/>
+                    <material name="Black"/>
+            </visual>
+            <collision>
+                    <geometry>
+                            <mesh filename="package://borunte_support/meshes/robotiq_gripper_collision.stl"/>
+                    </geometry>
+                    <origin rpy="0 0 0.0" xyz="0 0 0"/>
+            </collision>
+        </link>
         <joint name="${prefix}link_6-tool0" type="fixed">
-                <origin xyz="0 0 0" rpy="${pi} ${-pi/2.0} 0" />
                 <parent link="${prefix}link_6" />
                 <child link="${prefix}tool0" />
+                <axis xyz="0 0 1"/>
+                <origin xyz="0 0 0.030" rpy="${pi} ${pi} ${pi/2.0}" />
+        </joint>
+        <link name="${prefix}tool0_tip" />
+        <joint name="${prefix}tool0-tool0_tip" type="fixed">
+                <parent link="${prefix}tool0" />
+                <child link="${prefix}tool0_tip" />
+                <origin xyz="0 0 0.15" rpy="0 0 0" />
         </joint>
 </xacro:macro>

Commit message: borunte_robot: add adapter and camera frame

File: src/borunte_support/urdf/borunte_macro.xacro (robot description, xacro)
@@ -188,7 +188,21 @@
         </joint>
         <!-- ROS-Industrial 'flange' frame: attachment point for EEF models -->
-        <link name="${prefix}flange" />
+        <link name="${prefix}flange">
+            <visual>
+                    <geometry>
+                        <mesh filename="package://borunte_support/meshes/robotiq_adapter.stl"/>
+                    </geometry>
+                    <origin rpy="0 0 0.0" xyz="0 0 0"/>
+                    <material name="Black"/>
+            </visual>
+            <collision>
+                    <geometry>
+                            <mesh filename="package://borunte_support/meshes/robotiq_adapter_collision.stl"/>
+                    </geometry>
+                    <origin rpy="0 0 0.0" xyz="0 0 0"/>
+            </collision>
+        </link>
         <joint name="${prefix}joint_6-flange" type="fixed">
-                <origin xyz="0 0 0" rpy="0 0 0" />
+                <origin xyz="0 0 0.02" rpy="0 0 0" />
                 <parent link="${prefix}link_6" />
                 <child link="${prefix}flange" />
@@ -210,9 +224,9 @@
             </collision>
         </link>
-        <joint name="${prefix}link_6-tool0" type="fixed">
-                <parent link="${prefix}link_6" />
+        <joint name="${prefix}flange-tool0" type="fixed">
+                <parent link="${prefix}flange" />
                 <child link="${prefix}tool0" />
                 <axis xyz="0 0 1"/>
-                <origin xyz="0 0 0.030" rpy="${pi} ${pi} ${pi/2.0}" />
+                <origin xyz="0 0 0.0125" rpy="${pi} ${pi} ${pi/2.0}" />
         </joint>
         <link name="${prefix}tool0_tip" />
@@ -222,4 +236,11 @@
                 <origin xyz="0 0 0.15" rpy="0 0 0" />
         </joint>
+        <!-- Camera frame: location of wrist camera -->
+        <link name="${prefix}camera_link" />
+        <joint name="${prefix}flange-camera_link" type="fixed">
+          <origin xyz="0.06 0 0.03" rpy="0 0 0" />
+          <parent link="${prefix}flange" />
+          <child link="${prefix}camera_link" />
+        </joint>
 </xacro:macro>
 </robot>

Commit message: borunte_robot: rotate camera

File: src/borunte_support/urdf/borunte_macro.xacro (robot description, xacro)
@@ -239,5 +239,5 @@
         <link name="${prefix}camera_link" />
         <joint name="${prefix}flange-camera_link" type="fixed">
-          <origin xyz="0.06 0 0.03" rpy="0 0 0" />
+          <origin xyz="0.06 0 0.03" rpy="0 0 ${-pi/2.0}" />
           <parent link="${prefix}flange" />
           <child link="${prefix}camera_link" />

Commit message: borunte_support: fix orientation of camera

File: src/borunte_support/urdf/borunte_macro.xacro (robot description, xacro)
@@ -239,5 +239,5 @@
         <link name="${prefix}camera_link" />
         <joint name="${prefix}flange-camera_link" type="fixed">
-          <origin xyz="0.06 0 0.03" rpy="0 0 ${-pi/2.0}" />
+          <origin xyz="0.06 0 0.03" rpy="0 0 ${pi/2.0}" />
           <parent link="${prefix}flange" />
           <child link="${prefix}camera_link" />

Commit message: borunte_robot: increase joint limits

File: src/borunte_support/urdf/borunte_macro.xacro (robot description, xacro)
@@ -138,5 +138,5 @@
         <!-- joint list -->
 	<joint name="${prefix}joint_1" type="revolute">
-        	<limit effort="1000.0" lower="-2.967" upper="2.967" velocity="3.14"/>
+        	<limit effort="1000.0" lower="-3.076" upper="3.076" velocity="3.14"/>
                 <parent link="base_link"/>
                 <child link="link_1"/>
@@ -152,5 +152,5 @@
         </joint>
 	<joint name="${prefix}joint_3" type="revolute">
-                <limit effort="1000.0" lower="-1.571" upper="1.222" velocity="1.3"/>
+                <limit effort="1000.0" lower="-2.094" upper="1.570" velocity="1.3"/>
                 <parent link="link_2"/>
                 <child link="link_3"/>
@@ -166,5 +166,5 @@
         </joint>
         <joint name="${prefix}joint_5" type="revolute">
-                <limit effort="1000.0" lower="-1.571" upper="1.571" velocity="2.35"/>
+                <limit effort="1000.0" lower="-2.094" upper="2.094" velocity="2.35"/>
                 <parent link="link_4"/>
                 <child link="link_5"/>

Commit message: borunte_robot: fix joint positions

File: src/borunte_support/urdf/borunte_macro.xacro (robot description, xacro)
@@ -142,5 +142,5 @@
                 <child link="link_1"/>
 		<axis xyz="0 0 1"/>
-    		<origin rpy="0.0 0.0 0.0" xyz="0 0 0.271"/>
+    		<origin rpy="0.0 0.0 0.0" xyz="0 0 0.24"/>
         </joint>
 	<joint name="${prefix}joint_2" type="revolute">
@@ -149,5 +149,5 @@
                 <child link="link_2"/>
                 <axis xyz="0 1 0"/>
-                <origin rpy="0.0 0.0 0.0" xyz="0.07 0.095 0.1945"/>
+                <origin rpy="0.0 0.0 0.0" xyz="0.07 0.08 0.165"/>
         </joint>
 	<joint name="${prefix}joint_3" type="revolute">
@@ -159,5 +159,5 @@
         </joint>
 	<joint name="${prefix}joint_4" type="revolute">
-                <limit effort="1000.0" lower="-1.571" upper="1.571" velocity="2.0"/>
+                <limit effort="1000.0" lower="-2.094" upper="2.094" velocity="2.0"/>
                 <parent link="link_3"/>
                 <child link="link_4"/>
@@ -170,5 +170,5 @@
                 <child link="link_5"/>
                 <axis xyz="0 1 0"/>
-                <origin rpy="0.0 0.0 0.0" xyz="0.0 -0.0 0.3095"/>
+                <origin rpy="0.0 0.0 0.0" xyz="0.0 -0.0 0.31"/>
         </joint>
 	<joint name="${prefix}joint_6" type="revolute">
@@ -234,5 +234,5 @@
                 <parent link="${prefix}tool0" />
                 <child link="${prefix}tool0_tip" />
-                <origin xyz="0 0 0.15" rpy="0 0 0" />
+                <origin xyz="0 0 0.125" rpy="0 0 0" />
         </joint>
         <!-- Camera frame: location of wrist camera -->

Commit message: borunte: decrease joint 5 limit

File: src/borunte_support/urdf/borunte_macro.xacro (robot description, xacro)
@@ -166,5 +166,5 @@
         </joint>
         <joint name="${prefix}joint_5" type="revolute">
-                <limit effort="1000.0" lower="-2.094" upper="2.094" velocity="2.35"/>
+                <limit effort="1000.0" lower="-1.919" upper="2.094" velocity="2.35"/>
                 <parent link="link_4"/>
                 <child link="link_5"/>
@@ -234,5 +234,5 @@
                 <parent link="${prefix}tool0" />
                 <child link="${prefix}tool0_tip" />
-                <origin xyz="0 0 0.125" rpy="0 0 0" />
+                <origin xyz="0 0 0.15" rpy="0 0 0" />
         </joint>
         <!-- Camera frame: location of wrist camera -->

Commit message: borunte_robot: fix wrong dimensions in URDF

File: src/borunte_support/urdf/borunte_macro.xacro (robot description, xacro)
@@ -204,5 +204,5 @@
         </link>
         <joint name="${prefix}joint_6-flange" type="fixed">
-                <origin xyz="0 0 0.02" rpy="0 0 0" />
+                <origin xyz="0 0 0.015" rpy="0 0 0" />
                 <parent link="${prefix}link_6" />
                 <child link="${prefix}flange" />
@@ -228,5 +228,5 @@
                 <child link="${prefix}tool0" />
                 <axis xyz="0 0 1"/>
-                <origin xyz="0 0 0.0125" rpy="${pi} ${pi} ${pi/2.0}" />
+                <origin xyz="0 0 0.015" rpy="${pi} ${pi} ${pi/2.0}" />
         </joint>
         <link name="${prefix}tool0_tip" />

File: src/borunte_support/urdf/borunte_on_stand_macro.xacro (robot description, xacro)
@@ -3,5 +3,5 @@
 <xacro:macro name="borunte_on_stand_macro" params="prefix">
     <xacro:include filename="$(find borunte_support)/urdf/borunte_macro.xacro"/>
-    <xacro:borunte prefix="${prefix}" tool0_trans="0 0 0.15" tool0_rot="0 ${pi*1} 0"/>
+    <xacro:borunte prefix="${prefix}" tool0_trans="0 0 0.144" tool0_rot="0 ${pi*1} 0"/>
     <xacro:include filename="$(find borunte_support)/urdf/borunte_stand_macro.xacro"/>
     <xacro:borunte_stand prefix=""/>

Commit message: split Robotiq-Hand-E fingers and gripper

File: src/borunte_support/urdf/borunte_macro.xacro (robot description, xacro)
@@ -212,14 +212,14 @@
             <visual>
                     <geometry>
-                        <mesh filename="package://borunte_support/meshes/robotiq_gripper.stl"/>
-                    </geometry>
-                    <origin rpy="0 0 0.0" xyz="0 0 0"/>
-                    <material name="Black"/>
-            </visual>
-            <collision>
-                    <geometry>
-                            <mesh filename="package://borunte_support/meshes/robotiq_gripper_collision.stl"/>
-                    </geometry>
-                    <origin rpy="0 0 0.0" xyz="0 0 0"/>
+                        <mesh filename="package://borunte_support/meshes/robotiq_hand-e_gripper.stl"/>
+                    </geometry>
+                    <origin xyz="0 0 -0.005" rpy="0 0 0"/>
+                    <material name="Black"/>
+            </visual>
+            <collision>
+                    <geometry>
+                            <mesh filename="package://borunte_support/meshes/robotiq_hand-e_gripper_collision.stl"/>
+                    </geometry>
+                    <origin xyz="0 0 0" rpy="0 0 0"/>
             </collision>
         </link>
@@ -229,4 +229,46 @@
                 <axis xyz="0 0 1"/>
                 <origin xyz="0 0 0.015" rpy="${pi} ${pi} ${pi/2.0}" />
+        </joint>
+        <link name="${prefix}tool0_finger_left">
+            <visual>
+                    <geometry>
+                        <mesh filename="package://borunte_support/meshes/simple_grip_finger.stl"/>
+                    </geometry>
+                    <origin xyz="0 0 0" rpy="0 0 0"/>
+                    <material name="Black"/>
+            </visual>
+            <collision>
+                    <geometry>
+                            <mesh filename="package://borunte_support/meshes/simple_grip_finger_collision.stl"/>
+                    </geometry>
+                    <origin xyz="0 0 0" rpy="0 0 0.0"/>
+            </collision>
+        </link>
+        <joint name="${prefix}tool0-tool0_finger_left" type="fixed">
+                <parent link="${prefix}tool0" />
+                <child link="${prefix}tool0_finger_left" />
+                <axis xyz="0 0 1"/>
+                <origin xyz="0 0 0.095" rpy="0 0 ${pi/2.0}" />
+        </joint>
+        <link name="${prefix}tool0_finger_right">
+            <visual>
+                    <geometry>
+                        <mesh filename="package://borunte_support/meshes/simple_grip_finger.stl"/>
+                    </geometry>
+                    <origin xyz="0 0 0" rpy="0 0 0"/>
+                    <material name="Black"/>
+            </visual>
+            <collision>
+                    <geometry>
+                            <mesh filename="package://borunte_support/meshes/simple_grip_finger_collision.stl"/>
+                    </geometry>
+                    <origin xyz="0 0 0" rpy="0 0 0.0"/>
+            </collision>
+        </link>
+        <joint name="${prefix}tool0-tool0_finger_right" type="fixed">
+                <parent link="${prefix}tool0" />
+                <child link="${prefix}tool0_finger_right" />
+                <axis xyz="0 0 1"/>
+                <origin xyz="0 0 0.095" rpy="0 0 -${pi/2.0}" />
         </joint>
         <link name="${prefix}tool0_tip" />

Commit message: use tool0 instead of tool0_tip

File: src/borunte_support/urdf/borunte_macro.xacro (robot description, xacro)
@@ -204,10 +204,4 @@
       <child link="${prefix}tool0" />
     </joint>
-    <link name="${prefix}tool0_tip" />
-    <joint name="${prefix}tool0-tool0_tip" type="fixed">
-      <parent link="${prefix}tool0" />
-      <child link="${prefix}tool0_tip" />
-      <origin xyz="0 0 0" rpy="0 0 0" />
-    </joint>
   </xacro:macro>
 </robot>

Commit message: borunte_support: fix wrong dimensions

File: src/borunte_support/urdf/borunte_macro.xacro (robot description, xacro)
@@ -67,5 +67,5 @@
           <mesh filename="package://borunte_support/meshes/link_3.stl"/>
         </geometry>
-        <origin rpy="0.0 0 0.0" xyz="0 0 0"/>
+        <origin rpy="0.0 0 0.0" xyz="0 0.01 0"/>
         <material name="DarkRed"/>
       </visual>
@@ -74,5 +74,5 @@
           <mesh filename="package://borunte_support/meshes/link_3_collision.stl"/>
         </geometry>
-        <origin rpy="0.0 0 0.0" xyz="-0 0 0"/>
+        <origin rpy="0.0 0 0.0" xyz="0 0.01 0"/>
       </collision>
       <inertial>
@@ -151,5 +151,5 @@
       <child link="link_2"/>
       <axis xyz="0 1 0"/>
-      <origin rpy="0.0 0.0 0.0" xyz="0.07 0.08 0.165"/>
+      <origin rpy="0.0 0.0 0.0" xyz="0.07 0.09 0.165"/>
     </joint>
     <joint name="${prefix}joint_3" type="revolute">
@@ -165,5 +165,5 @@
       <child link="link_4"/>
       <axis xyz="0 0 1"/>
-      <origin rpy="0.0 0.0 0.0" xyz="-0.125 -0.1 0.095"/>
+      <origin rpy="0.0 0.0 0.0" xyz="-0.125 -0.09 0.075"/>
     </joint>
     <joint name="${prefix}joint_5" type="revolute">
@@ -179,5 +179,5 @@
       <child link="link_6"/>
       <axis xyz="0 0 1"/>
-      <origin rpy="0.0 0.0 0.0" xyz="0 0 0.089"/>
+      <origin rpy="0.0 0.0 0.0" xyz="0 0 0.104"/>
     </joint>
     <!-- ROS-Industrial 'base' frame: base_link to Fanuc World Coordinates transform -->

Commit message: borunte_support: decrease J2 limit to reduce config problems

File: src/borunte_support/urdf/borunte_macro.xacro (robot description, xacro)
@@ -147,5 +147,6 @@
     </joint>
     <joint name="${prefix}joint_2" type="revolute">
-      <limit effort="1000.0" lower="-1.74" upper="2.35" velocity="1.0"/>
+      <!-- actual limit -1.74, reduced to reduce config problems -->
+      <limit effort="1000.0" lower="-1.0" upper="2.35" velocity="1.0"/>
       <parent link="link_1"/>
       <child link="link_2"/>

Commit message: brounte_support: reduce rotation on joint 4

File: src/borunte_support/urdf/borunte_macro.xacro (robot description, xacro)
@@ -162,5 +162,6 @@
     </joint>
     <joint name="${prefix}joint_4" type="revolute">
-      <limit effort="1000.0" lower="-2.094" upper="2.094" velocity="2.0"/>
+      <!-- actual limit +-2.094, reduced to reduce config problems -->
+      <limit effort="1000.0" lower="${-pi/2.0}" upper="${pi/2.0}" velocity="2.0"/>
       <parent link="link_3"/>
       <child link="link_4"/>
