Commit message: move tool offset to xacro

File: src/borunte_support/urdf/borunte.xacro (robot description, xacro)
@@ -2,4 +2,4 @@
 <robot name="borunte" xmlns:xacro="http://www.ros.org/wiki/xacro">
 	<xacro:include filename="$(find borunte_support)/urdf/borunte_macro.xacro"/>
-	<xacro:borunte prefix=""/>
+	<xacro:borunte prefix="" tool0_trans="0 0 0.15" tool0_rot="0 0 0"/>
 </robot>

File: src/borunte_support/urdf/borunte_macro.xacro (robot description, xacro)
@@ -1,5 +1,5 @@
 <?xml version="1.0"?>
 <robot xmlns:xacro="http://www.ros.org/wiki/xacro">
-<xacro:macro name="borunte" params="prefix">
+<xacro:macro name="borunte" params="prefix tool0_trans tool0_rot">
         <!-- link list -->
 	<link name="${prefix}base_link">
@@ -234,5 +234,5 @@
                 <parent link="${prefix}tool0" />
                 <child link="${prefix}tool0_tip" />
-                <origin xyz="0 0 0.15" rpy="0 0 0" />
+                <origin xyz="${tool0_trans}" rpy="${tool0_rot}" />
         </joint>
         <!-- Camera frame: location of wrist camera -->
