Commit message: borunte_robot: rework URDF

File: src/borunte_support/urdf/borunte.xacro (robot description, xacro)
@@ -1,5 +1,5 @@
 <?xml version="1.0" ?>
 <robot name="borunte" xmlns:xacro="http://www.ros.org/wiki/xacro">
-	<xacro:include filename="$(find borunte_support)/urdf/borunte_macro.xacro"/>
-	<xacro:borunte prefix="" tool0_trans="0 0 0.15" tool0_rot="0 ${pi*1} 0"/>
+  <xacro:include filename="$(find borunte_support)/urdf/borunte_macro.xacro"/>
+  <xacro:borunte_macro prefix="" tool0_trans="0 0 0" tool0_rot="0 ${pi*1} 0"/>
 </robot>

File: src/borunte_support/urdf/borunte_macro.xacro (robot description, xacro)
@@ -1,288 +1,213 @@
 <?xml version="1.0"?>
 <robot xmlns:xacro="http://www.ros.org/wiki/xacro">
-<xacro:macro name="borunte" params="prefix tool0_trans tool0_rot">
-        <!-- link list -->
-	<link name="${prefix}base_link">
-                <visual>
-                        <geometry>
-                                <mesh filename="package://borunte_support/meshes/base_link.stl"/>
-                        </geometry>
-                        <origin rpy="0.0 0 0.0" xyz="0 0 0"/>
-                        <material name="Black">
-                                <color rgba="0.1 0.1 0.1 1.0"/>
-                        </material>
-                </visual>
-                <collision>
-                        <geometry>
-                                <mesh filename="package://borunte_support/meshes/base_link_collision.stl"/>
-                        </geometry>
-                        <origin rpy="0.0 0 0.0" xyz="0 0 0"/>
-                </collision>
-        </link>
-	<link name="${prefix}link_1">
-                <visual>
-                        <geometry>
-                                <mesh filename="package://borunte_support/meshes/link_1.stl"/>
-                        </geometry>
-                        <origin rpy="0.0 0 0.0" xyz="0 0 0"/>
-                        <material name="DarkRed">
-                                <color rgba="0.5 0.0 0.0 1.0"/>
-                        </material>
-                </visual>
-                <collision>
-                        <geometry>
-                                <mesh filename="package://borunte_support/meshes/link_1_collision.stl"/>
-                        </geometry>
-                        <origin rpy="0.0 0 0.0" xyz="0 0 0"/>
-                </collision>
-                <inertial>
-                        <mass value="100"/>
-                        <inertia ixx="1.0" ixy="0.0" ixz="0.0" iyy="1.0" iyz="0.0" izz="1.0"/>
-                </inertial>
-        </link>
-	<link name="${prefix}link_2">
-                <visual>
-                        <geometry>
-                                <mesh filename="package://borunte_support/meshes/link_2.stl"/>
-                        </geometry>
-                        <origin rpy="0.0 0 0.0" xyz="0 0 0"/>
-                        <material name="DarkRed"/>
-                </visual>
-                <collision>
-                        <geometry>
-                                <mesh filename="package://borunte_support/meshes/link_2_collision.stl"/>
-                        </geometry>
-                        <origin rpy="0.0 0 0.0" xyz="0 0 0"/>
-                </collision>
-                <inertial>
-                        <mass value="100"/>
-                        <inertia ixx="1.0" ixy="0.0" ixz="0.0" iyy="1.0" iyz="0.0" izz="1.0"/>
-                </inertial>
-        </link>
-	<link name="${prefix}link_3">
-                <visual>
-                        <geometry>
-                                <mesh filename="package://borunte_support/meshes/link_3.stl"/>
-                        </geometry>
-                        <origin rpy="0.0 0 0.0" xyz="0 0 0"/>
-                        <material name="DarkRed"/>
-                </visual>
-                <collision>
-                        <geometry>
-                                <mesh filename="package://borunte_support/meshes/link_3_collision.stl"/>
-                        </geometry>
-                        <origin rpy="0.0 0 0.0" xyz="-0 0 0"/>
-                </collision>
-                <inertial>
-                        <mass value="100"/>
-                        <inertia ixx="1.0" ixy="0.0" ixz="0.0" iyy="1.0" iyz="0.0" izz="1.0"/>
-                </inertial>
-        </link>
-	<link name="${prefix}link_4">
-                <visual>
-                        <geometry>
-                                <mesh filename="package://borunte_support/meshes/link_4.stl"/>
-                        </geometry>
-                        <origin rpy="0.0 0.0 0.0" xyz="0 0 0"/>
-                        <material name="DarkRed"/>
-                </visual>
-                <collision>
-                        <geometry>
-                                <mesh filename="package://borunte_support/meshes/link_4_collision.stl"/>
-                        </geometry>
-                        <origin rpy="0.0 0 0.0" xyz="0 0 0"/>
-                </collision>
-                <inertial>
-                        <mass value="100"/>
-                        <inertia ixx="1.0" ixy="0.0" ixz="0.0" iyy="1.0" iyz="0.0" izz="1.0"/>
-                </inertial>
-        </link>
-	<link name="${prefix}link_5">
-                <visual>
-                        <geometry>
-                                <mesh filename="package://borunte_support/meshes/link_5.stl"/>
-                        </geometry>
-                        <origin rpy="0 0 0" xyz="0 0 0"/>
-                        <material name="DarkRed"/>
-                </visual>
-                <collision>
-                        <geometry>
-                                <mesh filename="package://borunte_support/meshes/link_5_collision.stl"/>
-                        </geometry>
-                        <origin rpy="0 0 0" xyz="0 0 0"/>
-                </collision>
-                <inertial>
-                        <mass value="100"/>
-                        <inertia ixx="1.0" ixy="0.0" ixz="0.0" iyy="1.0" iyz="0.0" izz="1.0"/>
-                </inertial>
-        </link>
-	<link name="${prefix}link_6">
-                <visual>
-                        <geometry>
-                                <mesh filename="package://borunte_support/meshes/link_6.stl"/>
-                        </geometry>
-                        <origin rpy="0 0 0.0" xyz="0 0 0"/>
-                        <material name="DarkRed"/>
-                </visual>
-                <collision>
-                        <geometry>
-                                <mesh filename="package://borunte_support/meshes/link_6_collision.stl"/>
-                        </geometry>
-                        <origin rpy="0 0 0.0" xyz="0 0 0"/>
-                </collision>
-                <inertial>
-                        <mass value="100"/>
-                        <inertia ixx="1.0" ixy="0.0" ixz="0.0" iyy="1.0" iyz="0.0" izz="1.0"/>
-                </inertial>
-        </link>
-        <!-- joint list -->
-	<joint name="${prefix}joint_1" type="revolute">
-        	<limit effort="1000.0" lower="-3.076" upper="3.076" velocity="3.14"/>
-                <parent link="base_link"/>
-                <child link="link_1"/>
-		<axis xyz="0 0 1"/>
-    		<origin rpy="0.0 0.0 0.0" xyz="0 0 0.24"/>
-        </joint>
-	<joint name="${prefix}joint_2" type="revolute">
-		<limit effort="1000.0" lower="-1.74" upper="2.35" velocity="1.0"/>
-                <parent link="link_1"/>
-                <child link="link_2"/>
-                <axis xyz="0 1 0"/>
-                <origin rpy="0.0 0.0 0.0" xyz="0.07 0.08 0.165"/>
-        </joint>
-	<joint name="${prefix}joint_3" type="revolute">
-                <limit effort="1000.0" lower="-2.094" upper="1.570" velocity="1.3"/>
-                <parent link="link_2"/>
-                <child link="link_3"/>
-                <axis xyz="0 1 0"/>
-                <origin rpy="0.0 ${pi/2.0} 0.0" xyz="0.0 0.0 0.39"/>
-        </joint>
-	<joint name="${prefix}joint_4" type="revolute">
-                <limit effort="1000.0" lower="-2.094" upper="2.094" velocity="2.0"/>
-                <parent link="link_3"/>
-                <child link="link_4"/>
-                <axis xyz="0 0 1"/>
-                <origin rpy="0.0 0.0 0.0" xyz="-0.125 -0.1 0.095"/>
-        </joint>
-        <joint name="${prefix}joint_5" type="revolute">
-                <limit effort="1000.0" lower="-1.919" upper="2.094" velocity="2.35"/>
-                <parent link="link_4"/>
-                <child link="link_5"/>
-                <axis xyz="0 1 0"/>
-                <origin rpy="0.0 0.0 0.0" xyz="0.0 -0.0 0.31"/>
-        </joint>
-	<joint name="${prefix}joint_6" type="revolute">
-                <limit effort="1000.0" lower="${-pi}" upper="${pi}" velocity="2.35"/>
-                <parent link="link_5"/>
-                <child link="link_6"/>
-                <axis xyz="0 0 1"/>
-                <origin rpy="0.0 0.0 0.0" xyz="0 0 0.089"/>
-        </joint>
-        <!-- ROS-Industrial 'base' frame: base_link to Fanuc World Coordinates transform -->
-        <link name="${prefix}base" />
-        <joint name="${prefix}base_link-base" type="fixed">
-                <origin xyz="0 0 0" rpy="0 0 0"/>
-                <axis xyz="0 0 1"/>
-                <parent link="${prefix}base_link"/>
-                <child link="${prefix}base"/>
-        </joint>
-        <!-- ROS-Industrial 'flange' frame: attachment point for EEF models -->
-        <link name="${prefix}flange">
-            <visual>
-                    <geometry>
-                        <mesh filename="package://borunte_support/meshes/robotiq_adapter.stl"/>
-                    </geometry>
-                    <origin rpy="0 0 0.0" xyz="0 0 0"/>
-                    <material name="Black"/>
-            </visual>
-            <collision>
-                    <geometry>
-                            <mesh filename="package://borunte_support/meshes/robotiq_adapter_collision.stl"/>
-                    </geometry>
-                    <origin rpy="0 0 0.0" xyz="0 0 0"/>
-            </collision>
-        </link>
-        <joint name="${prefix}joint_6-flange" type="fixed">
-                <origin xyz="0 0 0.015" rpy="0 0 0" />
-                <parent link="${prefix}link_6" />
-                <child link="${prefix}flange" />
-        </joint>
-        <!-- ROS-Industrial 'tool0' frame: all-zeros tool frame -->
-        <link name="${prefix}tool0">
-            <visual>
-                    <geometry>
-                        <mesh filename="package://borunte_support/meshes/robotiq_hand-e_gripper.stl"/>
-                    </geometry>
-                    <origin xyz="0 0 -0.005" rpy="0 0 0"/>
-                    <material name="Black"/>
-            </visual>
-            <collision>
-                    <geometry>
-                            <mesh filename="package://borunte_support/meshes/robotiq_hand-e_gripper_collision.stl"/>
-                    </geometry>
-                    <origin xyz="0 0 0" rpy="0 0 0"/>
-            </collision>
-        </link>
-        <joint name="${prefix}flange-tool0" type="fixed">
-                <parent link="${prefix}flange" />
-                <child link="${prefix}tool0" />
-                <axis xyz="0 0 1"/>
-                <origin xyz="0 0 0.015" rpy="${pi} ${pi} ${pi/2.0}" />
-        </joint>
-        <link name="${prefix}tool0_finger_left">
-            <visual>
-                    <geometry>
-                        <mesh filename="package://borunte_support/meshes/simple_grip_finger.stl"/>
-                    </geometry>
-                    <origin xyz="0 0 0" rpy="0 0 0"/>
-                    <material name="Black"/>
-            </visual>
-            <collision>
-                    <geometry>
-                            <mesh filename="package://borunte_support/meshes/simple_grip_finger_collision.stl"/>
-                    </geometry>
-                    <origin xyz="0 0 0" rpy="0 0 0.0"/>
-            </collision>
-        </link>
-        <joint name="${prefix}tool0-tool0_finger_left" type="fixed">
-                <parent link="${prefix}tool0" />
-                <child link="${prefix}tool0_finger_left" />
-                <axis xyz="0 0 1"/>
-                <origin xyz="0 0 0.095" rpy="0 0 ${pi/2.0}" />
-        </joint>
-        <link name="${prefix}tool0_finger_right">
-            <visual>
-                    <geometry>
-                        <mesh filename="package://borunte_support/meshes/simple_grip_finger.stl"/>
-                    </geometry>
-                    <origin xyz="0 0 0" rpy="0 0 0"/>
-                    <material name="Black"/>
-            </visual>
-            <collision>
-                    <geometry>
-                            <mesh filename="package://borunte_support/meshes/simple_grip_finger_collision.stl"/>
-                    </geometry>
-                    <origin xyz="0 0 0" rpy="0 0 0.0"/>
-            </collision>
-        </link>
-        <joint name="${prefix}tool0-tool0_finger_right" type="fixed">
-                <parent link="${prefix}tool0" />
-                <child link="${prefix}tool0_finger_right" />
-                <axis xyz="0 0 1"/>
-                <origin xyz="0 0 0.095" rpy="0 0 -${pi/2.0}" />
-        </joint>
-        <link name="${prefix}tool0_tip" />
-        <joint name="${prefix}tool0-tool0_tip" type="fixed">
-                <parent link="${prefix}tool0" />
-                <child link="${prefix}tool0_tip" />
-                <origin xyz="${tool0_trans}" rpy="${tool0_rot}" />
-        </joint>
-        <!-- Camera frame: location of wrist camera -->
-        <link name="${prefix}camera_link" />
-        <joint name="${prefix}flange-camera_link" type="fixed">
-          <origin xyz="0.06 0 0.03" rpy="0 0 ${pi/2.0}" />
-          <parent link="${prefix}flange" />
-          <child link="${prefix}camera_link" />
-        </joint>
-</xacro:macro>
+  <xacro:macro name="borunte_macro" params="prefix tool0_trans tool0_rot">
+    <material name="Black">
+      <color rgba="0.1 0.1 0.1 1.0"/>
+    </material>
+    <material name="DarkRed">
+      <color rgba="0.5 0.0 0.0 1.0"/>
+    </material>
+    <!-- link list -->
+    <link name="${prefix}base_link">
+      <visual>
+        <geometry>
+          <mesh filename="package://borunte_support/meshes/base_link.stl"/>
+        </geometry>
+        <origin rpy="0.0 0 0.0" xyz="0 0 0"/>
+        <material name="Black"/>
+      </visual>
+      <collision>
+        <geometry>
+          <mesh filename="package://borunte_support/meshes/base_link_collision.stl"/>
+        </geometry>
+        <origin rpy="0.0 0 0.0" xyz="0 0 0"/>
+      </collision>
+    </link>
+    <link name="${prefix}link_1">
+      <visual>
+        <geometry>
+          <mesh filename="package://borunte_support/meshes/link_1.stl"/>
+        </geometry>
+        <origin rpy="0.0 0 0.0" xyz="0 0 0"/>
+        <material name="DarkRed"/>
+      </visual>
+      <collision>
+        <geometry>
+          <mesh filename="package://borunte_support/meshes/link_1_collision.stl"/>
+        </geometry>
+        <origin rpy="0.0 0 0.0" xyz="0 0 0"/>
+      </collision>
+      <inertial>
+        <mass value="100"/>
+        <inertia ixx="1.0" ixy="0.0" ixz="0.0" iyy="1.0" iyz="0.0" izz="1.0"/>
+      </inertial>
+    </link>
+    <link name="${prefix}link_2">
+      <visual>
+        <geometry>
+          <mesh filename="package://borunte_support/meshes/link_2.stl"/>
+        </geometry>
+        <origin rpy="0.0 0 0.0" xyz="0 0 0"/>
+        <material name="DarkRed"/>
+      </visual>
+      <collision>
+        <geometry>
+          <mesh filename="package://borunte_support/meshes/link_2_collision.stl"/>
+        </geometry>
+        <origin rpy="0.0 0 0.0" xyz="0 0 0"/>
+      </collision>
+      <inertial>
+        <mass value="100"/>
+        <inertia ixx="1.0" ixy="0.0" ixz="0.0" iyy="1.0" iyz="0.0" izz="1.0"/>
+      </inertial>
+    </link>
+    <link name="${prefix}link_3">
+      <visual>
+        <geometry>
+          <mesh filename="package://borunte_support/meshes/link_3.stl"/>
+        </geometry>
+        <origin rpy="0.0 0 0.0" xyz="0 0 0"/>
+        <material name="DarkRed"/>
+      </visual>
+      <collision>
+        <geometry>
+          <mesh filename="package://borunte_support/meshes/link_3_collision.stl"/>
+        </geometry>
+        <origin rpy="0.0 0 0.0" xyz="-0 0 0"/>
+      </collision>
+      <inertial>
+        <mass value="100"/>
+        <inertia ixx="1.0" ixy="0.0" ixz="0.0" iyy="1.0" iyz="0.0" izz="1.0"/>
+      </inertial>
+    </link>
+    <link name="${prefix}link_4">
+      <visual>
+        <geometry>
+          <mesh filename="package://borunte_support/meshes/link_4.stl"/>
+        </geometry>
+        <origin rpy="0.0 0.0 0.0" xyz="0 0 0"/>
+        <material name="DarkRed"/>
+      </visual>
+      <collision>
+        <geometry>
+          <mesh filename="package://borunte_support/meshes/link_4_collision.stl"/>
+        </geometry>
+        <origin rpy="0.0 0 0.0" xyz="0 0 0"/>
+      </collision>
+      <inertial>
+        <mass value="100"/>
+        <inertia ixx="1.0" ixy="0.0" ixz="0.0" iyy="1.0" iyz="0.0" izz="1.0"/>
+      </inertial>
+    </link>
+    <link name="${prefix}link_5">
+      <visual>
+        <geometry>
+          <mesh filename="package://borunte_support/meshes/link_5.stl"/>
+        </geometry>
+        <origin rpy="0 0 0" xyz="0 0 0"/>
+        <material name="DarkRed"/>
+      </visual>
+      <collision>
+        <geometry>
+          <mesh filename="package://borunte_support/meshes/link_5_collision.stl"/>
+        </geometry>
+        <origin rpy="0 0 0" xyz="0 0 0"/>
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
File: src/borunte_support/urdf/borunte_on_stand.xacro (robot description, xacro)
@@ -2,4 +2,4 @@
 <robot name="borunte_on_stand" xmlns:xacro="http://www.ros.org/wiki/xacro">
 	<xacro:include filename="$(find borunte_support)/urdf/borunte_on_stand_macro.xacro"/>
-	<xacro:borunte_on_stand_macro prefix=""/>
+	<xacro:borunte_on_stand_macro robotprefix="" standprefix="" tool="$(arg tool)"/>
 </robot>

File: src/borunte_support/urdf/borunte_on_stand_macro.xacro (robot description, xacro)
@@ -1,16 +1,22 @@
 <?xml version="1.0"?>
 <robot xmlns:xacro="http://www.ros.org/wiki/xacro">
-<xacro:macro name="borunte_on_stand_macro" params="prefix">
-    <xacro:include filename="$(find borunte_support)/urdf/borunte_macro.xacro"/>
-    <xacro:borunte prefix="${prefix}" tool0_trans="0 0 0.144" tool0_rot="0 ${pi*1} 0"/>
+  <xacro:macro name="borunte_on_stand_macro" params="robotprefix standprefix tool">
+    <xacro:if value="${tool == 'none'}">
+      <xacro:include filename="$(find borunte_support)/urdf/borunte_macro.xacro"/>
+      <xacro:borunte_macro prefix="${robotprefix}" tool0_trans="0 0 0" tool0_rot="0 ${pi*1} 0"/>
+    </xacro:if>
+    <xacro:if value="${tool == 'hand_e'}">
+      <xacro:include filename="$(find borunte_support)/urdf/borunte_hand_e_macro.xacro"/>
+      <xacro:borunte_hand_e_macro prefix="${robotprefix}" tool0_trans="0 0 0.159" tool0_rot="0 ${pi*1} 0"/>
+    </xacro:if>
     <xacro:include filename="$(find borunte_support)/urdf/borunte_stand_macro.xacro"/>
-    <xacro:borunte_stand prefix=""/>
+    <xacro:borunte_stand_macro prefix="${standprefix}"/>
     <!-- attach robot to stand flange -->
     <joint name="robot_attach_joint" type="fixed">
-        <parent link="borunte_stand_flange"/>
-        <child link="${prefix}base_link"/>
-        <axis xyz="0 0 0"/>
-        <origin rpy="0.0 0.0 0.0" xyz="0 0 0"/>
+      <parent link="borunte_stand_flange"/>
+      <child link="${robotprefix}base_link"/>
+      <axis xyz="0 0 0"/>
+      <origin rpy="0.0 0.0 0.0" xyz="0 0 0"/>
     </joint>
-</xacro:macro>
+  </xacro:macro>
 </robot>

File: src/borunte_support/urdf/borunte_stand_macro.xacro (robot description, xacro)
@@ -1,31 +1,31 @@
 <?xml version="1.0"?>
 <robot xmlns:xacro="http://www.ros.org/wiki/xacro">
-<xacro:macro name="borunte_stand" params="prefix">
-        <!-- link list  -->
-	    <link name="${prefix}borunte_stand_link">
-                <visual>
-                        <geometry>
-                                <mesh filename="package://borunte_support/meshes/borunte_carriage.stl"/>
-                        </geometry>
-                        <origin rpy="0.0 0 0.0" xyz="0 0 0"/>
-                        <material name="DarkGray">
-                                <color rgba="0.5 0.5 0.5 1.0"/>
-                        </material>
-                </visual>
-                <collision>
-                        <geometry>
-                                <mesh filename="package://borunte_support/meshes/borunte_carriage.stl"/>
-                        </geometry>
-                        <origin rpy="0.0 0 0.0" xyz="0 0 0.016"/>
-                </collision>
-        </link>
-        <!-- link the robot is going to be attached to -->
-        <link name="${prefix}borunte_stand_flange" />
-	    <joint name="${prefix}borunte_stand_joint" type="fixed">
-                <parent link="${prefix}borunte_stand_link"/>
-                <child link="${prefix}borunte_stand_flange"/>
-                <axis xyz="0 0 0"/>
-                <origin rpy="0.0 0.0 ${pi/4.0}" xyz="0.0 0.0 0.735"/>
-        </joint>
-</xacro:macro>
+  <xacro:macro name="borunte_stand_macro" params="prefix">
+    <!-- link list  -->
+    <link name="${prefix}borunte_stand_link">
+      <visual>
+        <geometry>
+          <mesh filename="package://borunte_support/meshes/borunte_carriage.stl"/>
+        </geometry>
+        <origin rpy="0.0 0 0.0" xyz="0 0 0"/>
+        <material name="DarkGray">
+          <color rgba="0.5 0.5 0.5 1.0"/>
+        </material>
+      </visual>
+      <collision>
+        <geometry>
+          <mesh filename="package://borunte_support/meshes/borunte_carriage.stl"/>
+        </geometry>
+        <origin rpy="0.0 0 0.0" xyz="0 0 0.016"/>
+      </collision>
+    </link>
+    <!-- link the robot is going to be attached to -->
+    <link name="${prefix}borunte_stand_flange" />
+    <joint name="${prefix}borunte_stand_joint" type="fixed">
+      <parent link="${prefix}borunte_stand_link"/>
+      <child link="${prefix}borunte_stand_flange"/>
+      <axis xyz="0 0 0"/>
+      <origin rpy="0.0 0.0 ${pi/4.0}" xyz="0.0 0.0 0.735"/>
+    </joint>
+  </xacro:macro>
 </robot>
