Commit message: borunte_support: move tool offset definition to tool macro

File: src/borunte_support/urdf/borunte.xacro (robot description, xacro)
@@ -1,5 +1,5 @@
 <?xml version="1.0" ?>
 <robot name="borunte" xmlns:xacro="http://www.ros.org/wiki/xacro">
-  <xacro:include filename="$(find borunte_support)/urdf/borunte_macro.xacro"/>
-  <xacro:borunte_macro prefix="" tool0_trans="0 0 0" tool0_rot="0 ${pi*1} 0"/>
+  <xacro:include filename="$(find borunte_support)/urdf/borunte_none_macro.xacro"/>
+  <xacro:borunte_none_macro prefix=""/>
 </robot>

File: src/borunte_support/urdf/borunte_hand_e.xacro (robot description, xacro)
@@ -2,4 +2,4 @@
 <robot name="borunte" xmlns:xacro="http://www.ros.org/wiki/xacro">
   <xacro:include filename="$(find borunte_support)/urdf/borunte_hand_e_macro.xacro"/>
-  <xacro:borunte_hand_e_macro prefix="" tool0_trans="0 0 0.159" tool0_rot="0 ${pi*1} 0"/>
+  <xacro:borunte_hand_e_macro prefix=""/>
 </robot>

File: src/borunte_support/urdf/borunte_hand_e_macro.xacro (robot description, xacro)
@@ -1,7 +1,7 @@
 <?xml version="1.0"?>
 <robot xmlns:xacro="http://www.ros.org/wiki/xacro">
-  <xacro:macro name="borunte_hand_e_macro" params="prefix tool0_trans tool0_rot">
+  <xacro:macro name="borunte_hand_e_macro" params="prefix">
     <xacro:include filename="$(find borunte_support)/urdf/borunte_macro.xacro"/>
-    <xacro:borunte_macro prefix="${prefix}" tool0_trans="${tool0_trans}" tool0_rot="${tool0_trans}"/>
+    <xacro:borunte_macro prefix="${prefix}"/>
     <xacro:include filename="$(find borunte_support)/urdf/robotiq_hand_e_macro.xacro"/>
     <xacro:robotiq_hand_e_macro prefix=""/>
@@ -14,4 +14,12 @@
       <child link="${prefix}borunte_robotiq_adapter" />
     </joint>
+    <!-- ROS-Industrial 'tool0' frame: all-zeros tool frame -->
+    <link name="${prefix}tool0" />
+    <joint name="${prefix}flange-tool0" type="fixed">
+      <!-- marker -->
+      <origin xyz="0 0 0.159" rpy="0 ${pi*1} 0" />
+      <parent link="${prefix}flange" />
+      <child link="${prefix}tool0" />
+    </joint>
   </xacro:macro>
 </robot>

File: src/borunte_support/urdf/borunte_macro.xacro (robot description, xacro)
@@ -1,5 +1,5 @@
 <?xml version="1.0"?>
 <robot xmlns:xacro="http://www.ros.org/wiki/xacro">
-  <xacro:macro name="borunte_macro" params="prefix tool0_trans tool0_rot">
+  <xacro:macro name="borunte_macro" params="prefix">
     <material name="Black">
       <color rgba="0.1 0.1 0.1 1.0"/>
@@ -196,12 +196,4 @@
       <child link="${prefix}flange" />
     </joint>
-    <!-- ROS-Industrial 'tool0' frame: all-zeros tool frame -->
-    <link name="${prefix}tool0" />
-    <joint name="${prefix}flange-tool0" type="fixed">
-      <!-- marker -->
-      <origin xyz="${tool0_trans}" rpy="${tool0_rot}" />
-      <parent link="${prefix}flange" />
-      <child link="${prefix}tool0" />
-    </joint>
   </xacro:macro>
 </robot>

File: src/borunte_support/urdf/borunte_on_stand_macro.xacro (robot description, xacro)
@@ -3,10 +3,10 @@
   <xacro:macro name="borunte_on_stand_macro" params="robotprefix standprefix tool">
     <xacro:if value="${tool == 'none'}">
-      <xacro:include filename="$(find borunte_support)/urdf/borunte_macro.xacro"/>
-      <xacro:borunte_macro prefix="${robotprefix}" tool0_trans="0 0 0" tool0_rot="0 ${pi*1} 0"/>
+      <xacro:include filename="$(find borunte_support)/urdf/borunte_none_macro.xacro"/>
+      <xacro:borunte_none_macro prefix="${robotprefix}"/>
     </xacro:if>
     <xacro:if value="${tool == 'hand_e'}">
       <xacro:include filename="$(find borunte_support)/urdf/borunte_hand_e_macro.xacro"/>
-      <xacro:borunte_hand_e_macro prefix="${robotprefix}" tool0_trans="0 0 0.159" tool0_rot="0 ${pi*1} 0"/>
+      <xacro:borunte_hand_e_macro prefix="${robotprefix}"/>
     </xacro:if>
     <xacro:include filename="$(find borunte_support)/urdf/borunte_stand_macro.xacro"/>

Commit message: borunte_support: cleanup xacro files

File: src/borunte_support/urdf/borunte.xacro (robot description, xacro)
@@ -1,4 +1,4 @@
 <?xml version="1.0" ?>
-<robot name="borunte" xmlns:xacro="http://www.ros.org/wiki/xacro">
+<robot name="borunte" xmlns:xacro="http://ros.org/wiki/xacro">
   <xacro:include filename="$(find borunte_support)/urdf/borunte_none_macro.xacro"/>
   <xacro:borunte_none_macro prefix=""/>

File: src/borunte_support/urdf/borunte_hand_e.xacro (robot description, xacro)
@@ -1,4 +1,4 @@
 <?xml version="1.0" ?>
-<robot name="borunte" xmlns:xacro="http://www.ros.org/wiki/xacro">
+<robot name="borunte" xmlns:xacro="http://ros.org/wiki/xacro">
   <xacro:include filename="$(find borunte_support)/urdf/borunte_hand_e_macro.xacro"/>
   <xacro:borunte_hand_e_macro prefix=""/>

File: src/borunte_support/urdf/borunte_hand_e_fish_fingers_macro.xacro (robot description, xacro)
@@ -1,4 +1,4 @@
 <?xml version="1.0"?>
-<robot xmlns:xacro="http://www.ros.org/wiki/xacro">
+<robot xmlns:xacro="http://ros.org/wiki/xacro">
   <xacro:macro name="borunte_hand_e_macro" params="prefix">
     <xacro:include filename="$(find borunte_support)/urdf/borunte_macro.xacro"/>

File: src/borunte_support/urdf/borunte_hand_e_macro.xacro (robot description, xacro)
@@ -1,4 +1,4 @@
 <?xml version="1.0"?>
-<robot xmlns:xacro="http://www.ros.org/wiki/xacro">
+<robot xmlns:xacro="http://ros.org/wiki/xacro">
   <xacro:macro name="borunte_hand_e_macro" params="prefix">
     <xacro:include filename="$(find borunte_support)/urdf/borunte_macro.xacro"/>

File: src/borunte_support/urdf/borunte_macro.xacro (robot description, xacro)
@@ -1,4 +1,4 @@
 <?xml version="1.0"?>
-<robot xmlns:xacro="http://www.ros.org/wiki/xacro">
+<robot xmlns:xacro="http://ros.org/wiki/xacro">
   <xacro:macro name="borunte_macro" params="prefix">
     <material name="Black">

File: src/borunte_support/urdf/borunte_none_macro.xacro (robot description, xacro)
@@ -1,4 +1,4 @@
 <?xml version="1.0"?>
-<robot xmlns:xacro="http://www.ros.org/wiki/xacro">
+<robot xmlns:xacro="http://ros.org/wiki/xacro">
   <xacro:macro name="borunte_none_macro" params="prefix">
     <xacro:include filename="$(find borunte_support)/urdf/borunte_macro.xacro"/>

File: src/borunte_support/urdf/borunte_on_stand.xacro (robot description, xacro)
@@ -1,4 +1,4 @@
 <?xml version="1.0" ?>
-<robot name="borunte_on_stand" xmlns:xacro="http://www.ros.org/wiki/xacro">
+<robot name="borunte_on_stand" xmlns:xacro="http://ros.org/wiki/xacro">
 	<xacro:include filename="$(find borunte_support)/urdf/borunte_on_stand_macro.xacro"/>
 	<xacro:borunte_on_stand_macro robotprefix="" standprefix="" tool="$(arg tool)"/>

File: src/borunte_support/urdf/borunte_on_stand_macro.xacro (robot description, xacro)
@@ -1,4 +1,4 @@
 <?xml version="1.0"?>
-<robot xmlns:xacro="http://www.ros.org/wiki/xacro">
+<robot xmlns:xacro="http://ros.org/wiki/xacro">
   <xacro:macro name="borunte_on_stand_macro" params="robotprefix standprefix tool">
     <xacro:if value="${tool == 'none'}">

File: src/borunte_support/urdf/borunte_stand_macro.xacro (robot description, xacro)
@@ -1,4 +1,4 @@
 <?xml version="1.0"?>
-<robot xmlns:xacro="http://www.ros.org/wiki/xacro">
+<robot xmlns:xacro="http://ros.org/wiki/xacro">
   <xacro:macro name="borunte_stand_macro" params="prefix">
     <!-- link list  -->

File: src/borunte_support/urdf/robotiq_hand_e.xacro (robot description, xacro)
@@ -1,4 +1,4 @@
 <?xml version="1.0" ?>
-<robot name="borunte" xmlns:xacro="http://www.ros.org/wiki/xacro">
+<robot name="borunte" xmlns:xacro="http://ros.org/wiki/xacro">
   <xacro:include filename="$(find borunte_support)/urdf/robotiq_hand_e_macro.xacro"/>
   <xacro:robotiq_hand_e_macro prefix=""/>

File: src/borunte_support/urdf/robotiq_hand_e_base_macro.xacro (robot description, xacro)
@@ -1,4 +1,4 @@
 <?xml version="1.0"?>
-<robot xmlns:xacro="http://www.ros.org/wiki/xacro">
+<robot xmlns:xacro="http://ros.org/wiki/xacro">
   <xacro:macro name="robotiq_hand_e_base_macro" params="prefix">
     <material name="Black_Aluminum">
@@ -8,5 +8,5 @@
       <color rgba="0.9 0.9 0.9 1.0"/>
     </material>
-      <link name="${prefix}borunte_robotiq_adapter">
+    <link name="${prefix}borunte_robotiq_adapter">
       <visual>
         <geometry>
@@ -44,5 +44,5 @@
       <origin xyz="0 0 0.015" rpy="${pi} ${pi} ${pi/2.0}" />
     </joint>
-        <!-- Camera frame: location of wrist camera -->
+    <!-- Camera frame: location of wrist camera -->
     <link name="${prefix}camera_link" />
     <joint name="${prefix}borunte_robotiq_adapter-camera_link" type="fixed">

File: src/borunte_support/urdf/robotiq_hand_e_fish_fingers_macro.xacro (robot description, xacro)
@@ -1,4 +1,4 @@
 <?xml version="1.0"?>
-<robot xmlns:xacro="http://www.ros.org/wiki/xacro">
+<robot xmlns:xacro="http://ros.org/wiki/xacro">
   <xacro:macro name="robotiq_hand_e_macro" params="prefix">
     <xacro:include filename="$(find borunte_support)/urdf/robotiq_hand_e_base_macro.xacro"/>

File: src/borunte_support/urdf/robotiq_hand_e_macro.xacro (robot description, xacro)
@@ -1,4 +1,4 @@
 <?xml version="1.0"?>
-<robot xmlns:xacro="http://www.ros.org/wiki/xacro">
+<robot xmlns:xacro="http://ros.org/wiki/xacro">
   <xacro:macro name="robotiq_hand_e_macro" params="prefix">
     <xacro:include filename="$(find borunte_support)/urdf/robotiq_hand_e_base_macro.xacro"/>

Commit message: borunte_robot: add alpha to colors and move world pose to top

File: src/borunte_support/urdf/borunte.xacro (robot description, xacro)
@@ -1,5 +1,13 @@
 <?xml version="1.0" ?>
 <robot name="borunte" xmlns:xacro="http://ros.org/wiki/xacro">
-  <xacro:include filename="$(find borunte_support)/urdf/borunte_none_macro.xacro"/>
-  <xacro:borunte_none_macro prefix=""/>
+    <xacro:include filename="$(find borunte_support)/urdf/borunte_none_macro.xacro"/>
+    <xacro:borunte_none_macro prefix=""/>
+    <!-- 'world' frame: default pose reference frame -->
+    <link name="world" />
+    <joint name="world-base_link" type="fixed">
+      <origin xyz="0 0 0" rpy="0 0 0"/>
+      <axis xyz="0 0 1"/>
+      <child link="world"/>
+      <parent link="base_link"/>
+    </joint>
 </robot>

File: src/borunte_support/urdf/borunte_ezgripper_gen2_plus_macro.xacro (robot description, xacro)
@@ -9,6 +9,6 @@
       <origin xyz="0 0 0.012" rpy="${pi} ${-pi/2.0} 0"/>
     </ezgripper_dual>
-    <material name="Black_Plastic">
-      <color rgba="0.1 0.1 0.1 1.0"/>
+    <material name="${prefix}Black_Plastic">
+      <color rgba="0.1 0.1 0.1 0.99"/>
     </material>
     <link name="${prefix}borunte_ezgripper_adapter">
@@ -18,5 +18,5 @@
         </geometry>
         <origin xyz="0 0 0" rpy="0 0 0" />
-        <material name="Black_Plastic"/>
+        <material name="${prefix}Black_Plastic"/>
       </visual>
       <collision>

File: src/borunte_support/urdf/borunte_hand_e.xacro (robot description, xacro)
@@ -1,5 +1,13 @@
 <?xml version="1.0" ?>
 <robot name="borunte" xmlns:xacro="http://ros.org/wiki/xacro">
-  <xacro:include filename="$(find borunte_support)/urdf/borunte_hand_e_macro.xacro"/>
-  <xacro:borunte_hand_e_macro prefix=""/>
+    <xacro:include filename="$(find borunte_support)/urdf/borunte_hand_e_macro.xacro"/>
+    <xacro:borunte_hand_e_macro prefix=""/>
+        <!-- 'world' frame: default pose reference frame -->
+    <link name="world" />
+    <joint name="world-base_link" type="fixed">
+      <origin xyz="0 0 0" rpy="0 0 0"/>
+      <axis xyz="0 0 1"/>
+      <child link="world"/>
+      <parent link="base_link"/>
+    </joint>
 </robot>

File: src/borunte_support/urdf/borunte_macro.xacro (robot description, xacro)
@@ -2,9 +2,9 @@
 <robot xmlns:xacro="http://ros.org/wiki/xacro">
   <xacro:macro name="borunte_macro" params="prefix">
-    <material name="Black">
-      <color rgba="0.1 0.1 0.1 1.0"/>
+    <material name="${prefix}Black">
+      <color rgba="0.1 0.1 0.1 0.99"/>
     </material>
-    <material name="DarkRed">
-      <color rgba="0.5 0.0 0.0 1.0"/>
+    <material name="${prefix}DarkRed">
+      <color rgba="0.5 0.0 0.0 0.99"/>
     </material>
     <!-- link list -->
@@ -15,5 +15,5 @@
         </geometry>
         <origin rpy="0.0 0 0.0" xyz="0 0 0"/>
-        <material name="Black"/>
+        <material name="${prefix}Black"/>
       </visual>
       <collision>
@@ -30,5 +30,5 @@
         </geometry>
         <origin rpy="0.0 0 0.0" xyz="0 0 0"/>
-        <material name="DarkRed"/>
+        <material name="${prefix}DarkRed"/>
       </visual>
       <collision>
@@ -49,5 +49,5 @@
         </geometry>
         <origin rpy="0.0 0 0.0" xyz="0 0 0"/>
-        <material name="DarkRed"/>
+        <material name="${prefix}DarkRed"/>
       </visual>
       <collision>
@@ -68,5 +68,5 @@
         </geometry>
         <origin rpy="0.0 0 0.0" xyz="0 0.01 0"/>
-        <material name="DarkRed"/>
+        <material name="${prefix}DarkRed"/>
       </visual>
       <collision>
@@ -87,5 +87,5 @@
         </geometry>
         <origin rpy="0.0 0.0 0.0" xyz="0 0 0"/>
-        <material name="DarkRed"/>
+        <material name="${prefix}DarkRed"/>
       </visual>
       <collision>
@@ -106,5 +106,5 @@
         </geometry>
         <origin rpy="0 0 0" xyz="0 0 0"/>
-        <material name="DarkRed"/>
+        <material name="${prefix}DarkRed"/>
       </visual>
       <collision>
@@ -125,5 +125,5 @@
         </geometry>
         <origin rpy="0 0 0.0" xyz="0 0 0"/>
-        <material name="DarkRed"/>
+        <material name="${prefix}DarkRed"/>
       </visual>
       <collision>

File: src/borunte_support/urdf/borunte_on_stand.xacro (robot description, xacro)
@@ -3,3 +3,11 @@
 	<xacro:include filename="$(find borunte_support)/urdf/borunte_on_stand_macro.xacro"/>
 	<xacro:borunte_on_stand_macro robotprefix="" standprefix="" tool="$(arg tool)"/>
+    <!-- 'world' frame: default pose reference frame -->
+    <link name="world" />
+    <joint name="world-borunte_stand_link" type="fixed">
+      <origin xyz="0 0 0" rpy="0 0 0"/>
+      <axis xyz="0 0 1"/>
+      <child link="world"/>
+      <parent link="borunte_stand_link"/>
+    </joint>
 </robot>

File: src/borunte_support/urdf/borunte_stand_macro.xacro (robot description, xacro)
@@ -2,6 +2,6 @@
 <robot xmlns:xacro="http://ros.org/wiki/xacro">
   <xacro:macro name="borunte_stand_macro" params="prefix">
-    <material name="DarkGray">
-      <color rgba="0.5 0.5 0.5 1.0"/>
+    <material name="${prefix}DarkGray">
+      <color rgba="0.5 0.5 0.5 0.75"/>
     </material>
     <!-- link list  -->
@@ -12,5 +12,5 @@
         </geometry>
         <origin rpy="0.0 0 0.0" xyz="0 0 0"/>
-        <material name="DarkGray"/>
+        <material name="${prefix}DarkGray"/>
       </visual>
       <collision>
@@ -21,12 +21,4 @@
       </collision>
     </link>
-    <!-- 'world' frame: default pose reference frame -->
-    <link name="${prefix}world" />
-    <joint name="${prefix}borunte_stand_link-world" type="fixed">
-      <origin xyz="0 0 0" rpy="0 0 0"/>
-      <axis xyz="0 0 1"/>
-      <parent link="${prefix}borunte_stand_link"/>
-      <child link="${prefix}world"/>
-    </joint>
     <!-- link the robot is going to be attached to -->
     <link name="${prefix}borunte_stand_flange" />

File: src/borunte_support/urdf/robotiq_hand_e_base_macro.xacro (robot description, xacro)
@@ -2,9 +2,9 @@
 <robot xmlns:xacro="http://ros.org/wiki/xacro">
   <xacro:macro name="robotiq_hand_e_base_macro" params="prefix">
-    <material name="Black_Aluminum">
-      <color rgba="0.1 0.1 0.1 1.0"/>
+    <material name="${prefix}Black_Aluminum">
+      <color rgba="0.1 0.1 0.1 0.99"/>
     </material>
-    <material name="White_Plastic">
-      <color rgba="0.9 0.9 0.9 1.0"/>
+    <material name="${prefix}White_Plastic">
+      <color rgba="0.9 0.9 0.9 0.99"/>
     </material>
     <link name="${prefix}borunte_robotiq_adapter">
@@ -14,5 +14,5 @@
         </geometry>
         <origin xyz="0 0 0" rpy="0 0 0" />
-        <material name="White_Plastic"/>
+        <material name="${prefix}White_Plastic"/>
       </visual>
       <collision>
@@ -29,5 +29,5 @@
         </geometry>
         <origin xyz="0 0 -0.003" rpy="0 0 0"/>
-        <material name="Black_Aluminum"/>
+        <material name="${prefix}Black_Aluminum"/>
       </visual>
       <collision>

File: src/borunte_support/urdf/robotiq_hand_e_fish_fingers_macro.xacro (robot description, xacro)
@@ -4,6 +4,6 @@
     <xacro:include filename="$(find borunte_support)/urdf/robotiq_hand_e_base_macro.xacro"/>
     <xacro:robotiq_hand_e_base_macro prefix="${prefix}"/>
-    <material name="Blue_Rubber">
-      <color rgba="0.1 0.1 1.0 1.0"/>
+    <material name="${prefix}Blue_Rubber">
+      <color rgba="0.1 0.1 1.0 0.99"/>
     </material>
     <link name="${prefix}fish_finger_adapter_left">
@@ -13,5 +13,5 @@
         </geometry>
         <origin xyz="0 0 0" rpy="0 0 0"/>
-        <material name="Black_Aluminum"/>
+        <material name="${prefix}Black_Aluminum"/>
       </visual>
       <collision>
@@ -34,5 +34,5 @@
         </geometry>
         <origin xyz="0 0 0" rpy="0 0 ${pi}"/>
-        <material name="Black_Aluminum"/>
+        <material name="${prefix}Black_Aluminum"/>
       </visual>
       <collision>
@@ -55,5 +55,5 @@
         </geometry>
         <origin xyz="0 0 0" rpy="0 0 0"/>
-        <material name="Black_Aluminum"/>
+        <material name="${prefix}Black_Aluminum"/>
       </visual>
       <collision>
@@ -76,5 +76,5 @@
         </geometry>
         <origin xyz="0 0 0" rpy="0 0 0"/>
-        <material name="Blue_Rubber"/>
+        <material name="${prefix}Blue_Rubber"/>
       </visual>
       <collision>
@@ -97,5 +97,5 @@
         </geometry>
         <origin xyz="0 0 0" rpy="0 0 0"/>
-        <material name="Black_Aluminum"/>
+        <material name="${prefix}Black_Aluminum"/>
       </visual>
       <collision>
@@ -118,5 +118,5 @@
         </geometry>
         <origin xyz="0 0 0" rpy="0 0 0"/>
-        <material name="Blue_Rubber"/>
+        <material name="${prefix}Blue_Rubber"/>
       </visual>
       <collision>

File: src/borunte_support/urdf/robotiq_hand_e_macro.xacro (robot description, xacro)
@@ -10,5 +10,5 @@
         </geometry>
         <origin xyz="0 0 0" rpy="0 0 0"/>
-        <material name="Black_Aluminum"/>
+        <material name="${prefix}Black_Aluminum"/>
       </visual>
       <collision>
@@ -31,5 +31,5 @@
         </geometry>
         <origin xyz="0 0 0" rpy="0 0 0"/>
-        <material name="Black_Aluminum"/>
+        <material name="${prefix}Black_Aluminum"/>
       </visual>
       <collision>
